Commit message: fixed rviz, allowed for multiple instances of the quantizer qubes

File: qube_description/urdf/qube.macro.xacro (robot description, xacro)
@@ -1,6 +1,70 @@
 <?xml version="1.0"?>
-<robot xmlns:xacro="http://www.ros.org/wiki/xacro" >
-	<xacro:macro name="qube">
-		Her ligger beskrivelsen av Quben
+<robot xmlns:xacro="http://www.ros.org/wiki/xacro">
+  <material name = "black">
+    <color rgba="0 0 0 1"/>
+  </material>
+  <material name = "red">
+    <color rgba="1 0 0 1"/>
+  </material>
+  <material name = "white">
+    <color rgba="1 1 1 1"/>
+  </material>
+	<xacro:macro name="qube_model" params="prefix base_x base_y base_z">
+		<xacro:property name="box_width" value="0.102"/>
+		<xacro:property name="angle_link_length" value="0.025"/>
+		<xacro:property name="angle_link_width" value="0.002"/>
+    <xacro:property name="angle_limit" value="3.14"/>
+    <xacro:property name="rotor_radius" value="0.025"/>
+    <xacro:property name="rotor_length" value="0.01"/>
+    <link name="${prefix}base_link"/>
+    <joint name="${prefix}base_joint" type="fixed">
+        <parent link="world"/>
+        <child link="${prefix}base_link"/>
+        <origin xyz="${base_x} ${base_y} ${base_z}" rpy="0 0 0"/>
+    </joint>
+		<link name="${prefix}stator_link">
+      <visual>
+        <geometry>
+          <box size="${box_width} ${box_width} ${box_width}"/>
+        </geometry>
+        <origin xyz="0 0 0" rpy="0 0 0"/>
+        <material name="black"/>
+      </visual>
+    </link>
+    <link name="${prefix}rotor_link">
+      <visual>
+        <geometry>
+          <cylinder length="${rotor_length}" radius="${rotor_radius}"/>
+        </geometry>
+        <origin xyz="0 0 0" rpy="0 0 0"/>
+        <material name="red"/>
+      </visual>
+    </link>
+    <link name="${prefix}angle_link">
+      <visual>
+        <geometry>
+          <box size="${angle_link_length} ${angle_link_width} ${angle_link_width}"/>
+        </geometry>
+        <origin xyz="0 0 0" rpy="0 0 0"/>
+        <material name="white"/>
+      </visual>
+    </link>
+    <joint name="${prefix}stator_joint" type="fixed">
+      <parent link="${prefix}base_link"/>
+      <child link="${prefix}stator_link"/>
+      <origin xyz="0 0 ${box_width/2}" rpy="0 0 0"/>
+    </joint>
+    <joint name="${prefix}angle_joint" type="revolute">
+      <parent link="${prefix}stator_link"/>
+      <child link="${prefix}rotor_link"/>
+      <origin xyz="0 0 ${box_width/2}" rpy="0 0 0"/>
+      <axis xyz="0 0 1"/>
+      <limit lower="-3.14" upper="3.14" effort="100.0" velocity="1.0"/>
+    </joint>
+    <joint name="${prefix}indicator_joint" type="fixed">
+      <parent link="${prefix}rotor_link"/>
+      <child link="${prefix}angle_link"/>
+      <origin xyz="0.0125 0 0.005" rpy="0 0 0"/>
+    </joint>
 	</xacro:macro>
 </robot>
